Commit message: car

File: demo_car/robots/demo_car.urdf (robot description, URDF)
Before this commit: robot damo_car, 3 links, 2 joints
Links:
- removed link wheel_L_Link
- removed link wheel_R_Link
- added link L_Link, mass 0.1; collision mesh filename=package://demo_car/meshes/L_Link.STL; visual mesh filename=package://demo_car/meshes/L_Link.STL
- added link R_Link, mass 0.1; collision mesh filename=package://demo_car/meshes/R_Link.STL; visual mesh filename=package://demo_car/meshes/R_Link.STL
- link base_link: mass 0.16184 -> 1; geometry collision mesh filename=package://demo_car/meshes/base_link.STL; visual mesh filename=package://demo_car/meshes/base_link.STL
Joints:
- removed joint wheel_L
- removed joint wheel_R
- added joint joint_L: type continuous, parent base_link, child L_Link, origin xyz=-0.051 0 0.0025 rpy=1.5708 1.5708 0, axis 0 -1 0
- added joint joint_R: type continuous, parent base_link, child R_Link, origin xyz=0.051 0 0.0025 rpy=1.5708 1.5708 0, axis 0 -1 0
